File: KH910_Power_Board Formatted/KH910_Power_Board_Formatted.kicad_sch (KiCad schematic)
At the start: 72 parts, among them P11 Conn_01x03_Pin, P8 Conn_01x02_Pin, P9 Conn_01x04_Pin, Q201 BD441, Q202 BD441, Q203 BC547, Q204 BD442, Q205 BC547, Q206 BD441, Q207 BC547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

Commit message: Created newly formatted schematic that is simplified to make analysis easier. Fixed duplicate P8 label on original schematic.
Connections:
- net 5v: now reaches 5v_P_N_to_Motherboard1.2 (Pin_2), C205.1, Q214.3 (E), R225.1, U201.3 (OUT), ZD204.1 (K)
- net P8_Pin_1: now reaches D203.1 (K), D204.2 (A), P8.1 (Pin_1), Q206.2 (C), Q208.2 (C)
- net P8_Pin_2: now reaches D201.1 (K), D202.2 (A), P8.2 (Pin_2), Q202.2 (C), Q204.2 (C)
- net at Q210.1 (C), ZD203.1 (K): now also R216.2; no longer R216.1
- net S-6_Pin_5: now reaches Q205.2 (B), R210.2, R214.2, S-6_Ribbon_Cable_to_Motherboard1.5 (Pin_5)
- net 16v DC Output: now reaches 15v_P_N_to_Motherboard1.1 (Pin_1), BZ1.1 (+), C201.1, D205.1 (K), D206.1 (K), D208.1 (K), Q201.2 (C), R202.2, R203.1
- net 16v DC Output: now also F201.2; no longer F201.1
- net S-6_Pin_2: now reaches BZ1.2 (-), D205.2 (A), S-6_Ribbon_Cable_to_Motherboard1.2 (Pin_2)
- net 15v_DC_Rectifier_Output: now reaches BR202.1 (+), C202.1, C204.2, Q210.2 (B)
- net 15v_DC_Rectifier_Output: now also R216.1; no longer R216.2, U201.1 (IN)
- net 10v ~AC: now reaches BR202.2, P9.4 (Pin_4)
- net 10v ~AC: now also F202.2, P9.3 (Pin_3)
- net S-6_Pin_1: now reaches C203.1, Q210.3 (E), S-6_Ribbon_Cable_to_Motherboard1.1 (Pin_1)
- net 12.2v ~AC: now reaches D206.2 (A), D207.1 (K), P9.1 (Pin_1)
- net 12.5v ~AC: now reaches F203.1, P9.2 (Pin_2)
- net S-6_Pin_3: now reaches Q214.1 (C), R227.2, S-6_Ribbon_Cable_to_Motherboard1.3 (Pin_3)
- net S-6_Pin_4: now reaches Q203.2 (B), R206.1, R211.2, S-6_Ribbon_Cable_to_Motherboard1.4 (Pin_4)
- net 16v DC Output (fused with F201): now reaches D202.1 (K), D204.1 (K), Q204.1 (E), Q208.1 (E)
- net 16v DC Output (fused with F201): now also F201.1; no longer F201.2
- net S-6_Pin_6: now reaches R213.2, R215.2, S-6_Ribbon_Cable_to_Motherboard1.6 (Pin_6)
- new net 15v_Rectifier_Output: U201.1 (IN)
- no-connect marks 0 -> 1
Other:
- title: Brother KH-910 5v-15v Internal Power Board -> Brother KH-910 5v-15v Internal Power Board (Formatted)
- moved on the sheet: 15v_P_N_to_Motherboard1, 5v_P_N_to_Motherboard1, BR202, BZ1, C201, C202, C203, C204, C205, D201, D202, D203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
