File: KH910_Power_Board_Formatted/KH910_Power_Board_Formatted.kicad_sch (KiCad schematic)
At the start: 72 parts, among them P11 Conn_01x03_Pin, P8 Conn_01x02_Pin, P9 Conn_01x04_Pin, Q201 BD441, Q202 BD441, Q203 BC547, Q204 BD442, Q205 BC547, Q206 BD441, Q207 BC547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

Commit message: Realized I messed up the P11 connector and had it flipped in the schematic, just fixed that in the formatted version.
Parts:
- removed P9: Conn_01x04_Pin, symbol Connector:Conn_01x04_Pin
- renumbered 5v_P_N_to_Motherboard1 to 5v_P_N_to_Motherboard
Connections:
- net 12.2v ~AC is gone; now on net AC: D206.2 (A), D207.1 (K)
- net 12.5v ~AC is gone; now on net AC: F203.1
- net 15v_Rectifier_Output is gone; now on net 15v_DC_Rectifier_Output: U201.1 (IN)
- net at P11.2 (Pin_2), POWER_LED1.2 (A), Q201.1 (E): now also P11.1 (Pin_1); no longer P11.3 (Pin_3)
- net 10v ~AC renamed AC
- net 5v renamed 5v DC
Other:
- note added: "P9 Output Pins"
- moved on the sheet: P11

Commit message: Reformatted the P8 motor circuit to be more like an H-Bridge to make the formatted schematic easier to read.
Connections:
- net at Q203.3 (E), R208.2: no longer Q206.3 (B)
- net at Q204.3 (B), R207.1: now also Q206.3 (B)
Other:
- moved on the sheet: 15v_P_N_to_Motherboard1, 5v_P_N_to_Motherboard, BR202, BZ1, C201, C202, C203, C204, C205, D201, D202, D203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
